Commit message: Add 3D LiDAR to robot URDF.

File: leo_description/urdf/macros.xacro (robot description, xacro)
@@ -157,4 +157,26 @@
     <link name="${link_prefix}camera_optical_frame"/>
     <link name="${link_prefix}imu_frame"/>
+    <link name="${link_prefix}lidar_base">
+    <visual>
+      <geometry>
+        <box size="0.075 0.075 0.05"/>
+      </geometry>
+      <material name="grey_color">
+        <color rgba="0.8 0.8 0.8 1"/>
+      </material>
+    </visual>
+    </link>
+    <!-- LiDAR Visuals -->
+    <link name="${link_prefix}lidar_sphere">
+    <visual>
+      <geometry>
+        <sphere radius="0.025"/>
+      </geometry>
+      <material name="blue_color">
+        <color rgba="0.4 0.4 0.9 1"/>
+      </material>
+    </visual>
+    </link>
+    <link name="${link_prefix}livox_frame"/>
     <!-- JOINTS -->
     <xacro:if value="${footprint_link}">
@@ -262,4 +284,20 @@
       <child link="${link_prefix}imu_frame"/>
     </joint>
+    <!-- LiDAR joints -->
+    <joint name="${joint_prefix}lidar_base_joint" type="fixed">
+      <origin xyz="0.04 0 0" rpy="0 0 0"/>
+      <parent link="${link_prefix}base_link"/>
+      <child link="${link_prefix}lidar_base"/>
+    </joint>
+    <joint name="${joint_prefix}lidar_sphere_joint" type="fixed">
+      <origin xyz="0 0 0.02" rpy="0 0 0"/>
+      <parent link="${link_prefix}lidar_base"/>
+      <child link="${link_prefix}lidar_sphere"/>
+    </joint>
+    <joint name="${joint_prefix}lidar_joint" type="fixed">
+      <origin xyz="0 0 0.02" rpy="0 0 0"/>
+      <parent link="${link_prefix}lidar_sphere"/>
+      <child link="${link_prefix}livox_frame"/>
+    </joint>
   </xacro:macro>
   <!-- LEO GAZEBO -->
@@ -420,4 +458,40 @@
         </surface>
       </collision>
+    </gazebo>
+    <!-- 3D LiDAR -->
+    <gazebo reference="${link_prefix}livox_frame">
+      <sensor name="gpu_lidar" type="gpu_lidar">
+        <pose>0 0 0 0 0 0</pose>
+        <topic>livox/lidar</topic>
+        <update_rate>10</update_rate>
+        <visualize>true</visualize>
+        <ray>
+          <scan>
+            <horizontal>
+              <samples>640</samples>
+              <resolution>1</resolution>
+              <min_angle>-3.141592</min_angle>
+              <max_angle>3.141592</max_angle>
+            </horizontal>
+            <vertical>
+                <samples>40</samples>
+                <resolution>1</resolution>
+                <min_angle>-0.122173</min_angle>
+                <max_angle>0.9075712</max_angle>
+            </vertical>
+          </scan>
+          <range>
+            <min>0.1</min>
+            <max>20.0</max>
+            <resolution>0.01</resolution>
+          </range>
+          <noise>
+            <type>gaussian</type>
+            <mean>0.0</mean>
+            <stddev>0.01</stddev>
+          </noise>
+        </ray>
+        <ignition_frame_id>${link_prefix}livox_frame</ignition_frame_id>
+      </sensor>
     </gazebo>
     <!-- camera -->

Commit message: commit for the leo_common submodule

File: leo_description/urdf/macros.xacro (robot description, xacro)
@@ -198,6 +198,6 @@
       <child link="${link_prefix}rocker_L_link"/>
       <axis xyz="0 1 0"/>
-      <limit effort="100.0" lower="-0.24" upper="0.24" velocity="100.0"/>
-      <dynamics friction="1.0" damping="0.1"/>
+      <limit effort="100.0" lower="-5.0" upper="5.0" velocity="100.0"/>
+      <dynamics friction="1.0" damping="0.01"/>
     </joint>
     <joint name="${joint_prefix}rocker_R_joint" type="${rockers_joint_type}">
@@ -206,6 +206,6 @@
       <child link="${link_prefix}rocker_R_link"/>
       <axis xyz="0 1 0"/>
-      <limit effort="100.0" lower="-0.24" upper="0.24" velocity="100.0"/>
-      <dynamics friction="1.0" damping="0.1"/>
+      <limit effort="100.0" lower="-5.0" upper="5.0" velocity="100.0"/>
+      <dynamics friction="1.0" damping="0.01"/>
       <mimic joint="rocker_L_joint"/>
     </joint>
@@ -220,6 +220,6 @@
       <child link="${link_prefix}wheel_FL_link"/>
       <axis xyz="0 -1 0"/>
-      <limit effort="2.0" velocity="6.0"/>
-      <dynamics friction="0.3125" damping="0.1"/>
+      <limit effort="40.0" velocity="100.0"/>
+      <dynamics friction="0.3125" damping="0.01"/>
     </joint>
     <joint name="${joint_prefix}wheel_RL_joint" type="continuous">
@@ -233,6 +233,6 @@
       <child link="${link_prefix}wheel_RL_link"/>
       <axis xyz="0 -1 0"/>
-      <limit effort="2.0" velocity="6.0"/>
-      <dynamics friction="0.3125" damping="0.1"/>
+      <limit effort="40.0" velocity="100.0"/>
+      <dynamics friction="0.3125" damping="0.01"/>
     </joint>
     <joint name="${joint_prefix}wheel_FR_joint" type="continuous">
@@ -246,6 +246,6 @@
       <child link="${link_prefix}wheel_FR_link"/>
       <axis xyz="0 1 0"/>
-      <limit effort="2.0" velocity="6.0"/>
-      <dynamics friction="0.3125" damping="0.1"/>
+      <limit effort="40.0" velocity="100.0"/>
+      <dynamics friction="0.3125" damping="0.01"/>
     </joint>
     <joint name="${joint_prefix}wheel_RR_joint" type="continuous">
@@ -259,6 +259,6 @@
       <child link="${link_prefix}wheel_RR_link"/>
       <axis xyz="0 1 0"/>
-      <limit effort="2.0" velocity="6.0"/>
-      <dynamics friction="0.3125" damping="0.1"/>
+      <limit effort="40.0" velocity="100.0"/>
+      <dynamics friction="0.3125" damping="0.01"/>
     </joint>
     <xacro:if value="${default_antenna}">
@@ -386,11 +386,11 @@
               <mu>1</mu>
               <mu2>1</mu2>
-              <slip1>0.035</slip1>
+              <slip1>0</slip1>
               <slip2>0</slip2>
               <fdir1>0 0 1</fdir1>
             </ode>
             <bullet>
-              <friction>1</friction>
-              <friction2>1</friction2>
+              <friction>10</friction>
+              <friction2>10</friction2>
               <rolling_friction>0.1</rolling_friction>
             </bullet>
@@ -406,11 +406,11 @@
               <mu>1</mu>
               <mu2>1</mu2>
-              <slip1>0.035</slip1>
+              <slip1>0</slip1>
               <slip2>0</slip2>
               <fdir1>0 0 1</fdir1>
             </ode>
             <bullet>
-              <friction>1</friction>
-              <friction2>1</friction2>
+              <friction>10</friction>
+              <friction2>10</friction2>
               <rolling_friction>0.1</rolling_friction>
             </bullet>
@@ -426,11 +426,11 @@
               <mu>1</mu>
               <mu2>1</mu2>
-              <slip1>0.035</slip1>
+              <slip1>0</slip1>
               <slip2>0</slip2>
               <fdir1>0 0 1</fdir1>
             </ode>
             <bullet>
-              <friction>1</friction>
-              <friction2>1</friction2>
+              <friction>10</friction>
+              <friction2>10</friction2>
               <rolling_friction>0.1</rolling_friction>
             </bullet>
@@ -446,11 +446,11 @@
               <mu>1</mu>
               <mu2>1</mu2>
-              <slip1>0.035</slip1>
+              <slip1>0</slip1>
               <slip2>0</slip2>
               <fdir1>0 0 1</fdir1>
             </ode>
             <bullet>
-              <friction>1</friction>
-              <friction2>1</friction2>
+              <friction>10</friction>
+              <friction2>10</friction2>
               <rolling_friction>0.1</rolling_friction>
             </bullet>
@@ -547,4 +547,11 @@
         name="ignition::gazebo::systems::Imu">
       </plugin>
+      <plugin
+          filename="ignition-gazebo-pose-publisher-system"
+          name="ignition::gazebo::systems::PosePublisher">
+          <publish_link_pose>false</publish_link_pose>
+          <publish_nested_model_pose>true</publish_nested_model_pose>
+          <update_frequency>20</update_frequency>
+      </plugin>
     </gazebo>
     <gazebo reference="${link_prefix}imu_frame">
@@ -567,6 +574,6 @@
         <wheel_separation>0.358</wheel_separation>
         <wheel_radius>0.0625</wheel_radius>
-        <!-- <frame_id>odom</frame_id> --> <!-- Change frame names to avoid odom in TF tree -->
-        <frame_id>not_connected_odom</frame_id>
+        <!-- <frame_id>odom</frame_id>  -->
+        <frame_id>not_connected_odom</frame_id>  Change frame names to avoid odom in TF tree
         <!-- <child_frame_id>${link_prefix}base_footprint</child_frame_id> -->
         <child_frame_id>${link_prefix}not_connected_base_footprint</child_frame_id>
